File: mains/mains_bottom.brd (EAGLE design)
At the start: 39.3 x 106.5 mm, 85 parts, among them IC1 OPA4134D, IC2 OPA4134D, IC3 OPA2134UA, U1 TL074_SMD

Commit message: Fix!
Parts:
- R21, R22: value 22K -> 3.9K
Changed lines of the file:
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@@
 <attribute name="NAME" x="38.035" y="59.635" size="1.27" layer="25" rot="R270"/>
 </element>
-<element name="R22" library="resistor" library_urn="urn:adsk.eagle:library:348" package="R0603" package3d_urn="urn:adsk.eagle:package:26057/1" value="22K" x="24" y="62" smashed="yes" rot="R270">
+<element name="R22" library="resistor" library_urn="urn:adsk.eagle:library:348" package="R0603" package3d_urn="urn:adsk.eagle:package:26057/1" value="3.9K" x="24" y="62" smashed="yes" rot="R270">
 <attribute name="NAME" x="23.335" y="63.635" size="0.6096" layer="25"/>
 </element>
-<element name="R21" library="resistor" library_urn="urn:adsk.eagle:library:348" package="R0603" package3d_urn="urn:adsk.eagle:package:26057/1" value="22K" x="38" y="62" smashed="yes" rot="R270">
+<element name="R21" library="resistor" library_urn="urn:adsk.eagle:library:348" package="R0603" package3d_urn="urn:adsk.eagle:package:26057/1" value="3.9K" x="38" y="62" smashed="yes" rot="R270">
 <attribute name="NAME" x="37.435" y="63.635" size="0.6096" layer="25"/>
 </element>
