File: mains/mains_top.brd (EAGLE design)
At the start: 39.3 x 66.1 mm, 51 parts

Commit message: Fix!
Parts:
- moved POT_CUE 4.00 mm to (7.00, 74.0)
- moved POT_MAIN 4.00 mm to (33.0, 74.0)
Routing:
- net N$21: track 32.2 -> 25.5 mm
- net N$41: track 38.6 -> 32.2 mm
- net N$19: track 18.8 -> 15.0 mm
- net N$14: track 22.1 -> 18.3 mm
- net N$46: track 17.8 -> 14.2 mm
- net N$23: track 10.1 -> 6.63 mm
- net N$24: track 9.30 -> 5.79 mm
- net N$20: track 25.1 -> 22.0 mm
Changed lines of the file:
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@@
 </autorouter>
 <elements>
-<element name="POT_CUE" library="MusicThingModular" package="DUAL_9MM_SNAP-IN_POT" value="A50K" x="7" y="70"/>
-<element name="POT_MAIN" library="MusicThingModular" package="DUAL_9MM_SNAP-IN_POT" value="A50K" x="33" y="70" smashed="yes">
-<attribute name="NAME" x="29.19" y="72.54" size="1.0668" layer="25"/>
-<attribute name="VALUE" x="29.19" y="66.19" size="1.27" layer="27"/>
+<element name="POT_CUE" library="MusicThingModular" package="DUAL_9MM_SNAP-IN_POT" value="A50K" x="7" y="74"/>
+<element name="POT_MAIN" library="MusicThingModular" package="DUAL_9MM_SNAP-IN_POT" value="A50K" x="33" y="74" smashed="yes">
+<attribute name="NAME" x="29.19" y="76.54" size="1.0668" layer="25"/>
+<attribute name="VALUE" x="29.19" y="70.19" size="1.27" layer="27"/>
 </element>
 <element name="POT_HP" library="MusicThingModular" package="DUAL_9MM_SNAP-IN_POT" value="A50K" x="7" y="52"/>
@@
 <contactref element="C8" pad="2"/>
 <wire x1="35.7134" y1="73.2599625" x2="35.7134" y2="74.7400375" width="0.1524" layer="1"/>
-<wire x1="36.02" y1="64.98" x2="35.5" y2="60.46" width="0.1524" layer="1"/>
+<wire x1="36.02" y1="64.98" x2="35.5" y2="64.46" width="0.1524" layer="1"/>
 <wire x1="38.575" y1="80.3" x2="38.575" y2="77.6016375" width="0.1524" layer="1"/>
 <wire x1="38.575" y1="77.6016375" x2="35.7134" y2="74.7400375" width="0.1524" layer="1"/>
@@
 <contactref element="C6" pad="2"/>
 <wire x1="5.125" y1="80.2" x2="9" y2="76.325" width="0.1524" layer="1"/>
-<wire x1="9" y1="67.5" x2="9.5" y2="63" width="0.1524" layer="1"/>
+<wire x1="9" y1="67.5" x2="9.5" y2="67" width="0.1524" layer="1"/>
 <wire x1="9" y1="76.325" x2="9" y2="67.5" width="0.1524" layer="1"/>
 </signal>
@@
 <wire x1="5.9464" y1="64.02358125" x2="6.56358125" y2="63.4064" width="0.1524" layer="1"/>
 <wire x1="6.56358125" y1="63.4064" x2="7.43641875" y2="63.4064" width="0.1524" layer="1"/>
-<wire x1="8.49001875" y1="64.46" x2="9.5" y2="60.46" width="0.1524" layer="1"/>
+<wire x1="8.49001875" y1="64.46" x2="9.5" y2="64.46" width="0.1524" layer="1"/>
 <wire x1="7.43641875" y1="63.4064" x2="8.49001875" y2="64.46" width="0.1524" layer="1"/>
 <wire x1="2.125" y1="79.24276875" x2="5.9464" y2="75.42136875" width="0.1524" layer="1"/>
@@
 <contactref element="POT_MAIN" pad="2B"/>
 <contactref element="R6" pad="1"/>
-<wire x1="33" y1="60.46" x2="32.4732875" y2="64.46" width="0.1524" layer="1"/>
+<wire x1="33" y1="64.46" x2="32.4732875" y2="64.46" width="0.1524" layer="1"/>
 <wire x1="32.4732875" y1="64.46" x2="31.4196875" y2="65.5136" width="0.1524" layer="1"/>
 <wire x1="28.3364" y1="65.5136" x2="27.85" y2="66" width="0.1524" layer="1"/>
@@
 <wire x1="31.4196875" y1="65.9464" x2="29.5803125" y2="65.9464" width="0.1524" layer="1"/>
 <wire x1="29.5803125" y1="65.9464" x2="29.4464" y2="66.0803125" width="0.1524" layer="1"/>
-<wire x1="33" y1="63" x2="32.4732875" y2="67" width="0.1524" layer="1"/>
+<wire x1="33" y1="67" x2="32.4732875" y2="67" width="0.1524" layer="1"/>
 <wire x1="29.4464" y1="66.0803125" x2="29.4464" y2="66.4036" width="0.1524" layer="1"/>
 <wire x1="32.4732875" y1="67" x2="31.4196875" y2="65.9464" width="0.1524" layer="1"/>
@@
 <contactref element="POT_CUE" pad="2"/>
 <contactref element="R7" pad="1"/>
-<wire x1="7" y1="63" x2="10.5" y2="70.5" width="0.1524" layer="16"/>
-<wire x1="10.5" y1="70.5" x2="12.2134" y2="72.2134" width="0.1524" layer="16"/>
+<wire x1="7" y1="67" x2="12.2134" y2="72.2134" width="0.1524" layer="16"/>
 <wire x1="18.9332" y1="78.9818875" x2="19.5581125" y2="79.6068" width="0.1524" layer="16"/>
 <wire x1="19.5581125" y1="79.6068" x2="20.4418875" y2="79.6068" width="0.1524" layer="16"/>
@@
 <wire x1="9.93641875" y1="65.9464" x2="9.06358125" y2="65.9464" width="0.1524" layer="1"/>
 <wire x1="12.15" y1="67" x2="10.99001875" y2="67" width="0.1524" layer="1"/>
-<wire x1="8.00998125" y1="67" x2="7" y2="63" width="0.1524" layer="1"/>
+<wire x1="8.00998125" y1="67" x2="7" y2="67" width="0.1524" layer="1"/>
 <wire x1="10.99001875" y1="67" x2="9.93641875" y2="65.9464" width="0.1524" layer="1"/>
 <wire x1="9.06358125" y1="65.9464" x2="8.00998125" y2="67" width="0.1524" layer="1"/>
@@
 <contactref element="S1" pad="2"/>
 <wire x1="8.4464" y1="67.43641875" x2="9.06358125" y2="68.0536" width="0.1524" layer="16"/>
-<wire x1="7" y1="60.46" x2="8.4464" y2="65.9064" width="0.1524" layer="16"/>
+<wire x1="7" y1="64.46" x2="8.4464" y2="65.9064" width="0.1524" layer="16"/>
 <wire x1="8.4464" y1="65.9064" x2="8.4464" y2="67.43641875" width="0.1524" layer="16"/>
 <wire x1="9.06358125" y1="68.0536" x2="9.5136" y2="68.0536" width="0.1524" layer="16"/>
 <wire x1="9.5136" y1="68.0536" x2="20" y2="78.54" width="0.1524" layer="16"/>
 <wire x1="9.06358125" y1="65.5136" x2="9.93641875" y2="65.5136" width="0.1524" layer="1"/>
-<wire x1="7" y1="60.46" x2="8.00998125" y2="64.46" width="0.1524" layer="1"/>
+<wire x1="7" y1="64.46" x2="8.00998125" y2="64.46" width="0.1524" layer="1"/>
 <wire x1="8.00998125" y1="64.46" x2="9.06358125" y2="65.5136" width="0.1524" layer="1"/>
 <wire x1="9.93641875" y1="65.5136" x2="10.45001875" y2="65" width="0.1524" layer="1"/>
@@
 <wire x1="33.425" y1="80.3" x2="33.425" y2="72.03269375" width="0.1524" layer="1"/>
 <wire x1="33.425" y1="72.03269375" x2="34.3584" y2="71.09929375" width="0.1524" layer="1"/>
-<wire x1="34.3584" y1="68.1416" x2="35.5" y2="63" width="0.1524" layer="1"/>
+<wire x1="34.3584" y1="68.1416" x2="35.5" y2="67" width="0.1524" layer="1"/>
 <wire x1="34.3584" y1="71.09929375" x2="34.3584" y2="68.1416" width="0.1524" layer="1"/>
 </signal>
